Commit message: Tighten base joint limits: ±3m xy, ±π yaw
Was: ±20m xy, ±2π yaw — caused wild base motion in planning
Now: ±3m xy, ±π yaw — more practical for kitchen-scale environments

File: tidyverse.urdf (robot description, URDF)
Before this commit: robot tidyverse, 25 links, 24 joints
Joints:
- joint base_x_joint: limit lower=-20 upper=20 effort=600 velocity=1.0 -> lower=-3 upper=3 effort=600 velocity=1.0
- joint base_y_joint: limit lower=-20 upper=20 effort=600 velocity=1.0 -> lower=-3 upper=3 effort=600 velocity=1.0
- joint base_yaw_joint: limit lower=-6.28318 upper=6.28318 effort=600 velocity=1.5 -> lower=-3.14159 upper=3.14159 effort=600 velocity=1.5

Commit message: Replace base collision STL (150K tris) with box approximation
Box: 0.733 x 0.523 x 0.606m, centered at (-0.198, 0, 0.309) in base_link frame.
Matches bounding box of original base_col.stl mesh.
Visual mesh unchanged (still uses base_vis.stl for rendering).
Should dramatically speed up collision checking in SapienPlanner.

File: tidyverse.urdf (robot description, URDF)
Before this commit: robot tidyverse, 25 links, 24 joints
Links:
- link base_link: geometry collision box size=0.733 0.523 0.606; visual mesh filename=tidyverse_base/base_vis.stl
